File: MRM5-Sensor/MRM5-Sensor.kicad_pcb (KiCad board)
At the start: 2 copper layers, 50 x 25 mm, 12 parts, among them J1 1989447, J2 Conn_01x02_Socket, J3 Conn_01x02_Socket, J4 Conn_01x02_Socket, J5 Conn_01x02_Socket, P1 AC_L, P2 AC_N, T1 ZMPT107-1

Commit message: MRM5-tester added
Parts:
- moved P2 7.86 mm to (138.7, 85.6)
- moved R2 4.94 mm to (138.7, 81.0), turned to 90 degrees
- moved P1 4.73 mm to (123.4, 85.6)
- moved R1 4.04 mm to (123.4, 81.0), turned to 90 degrees
- moved J1 3.25 mm to (118.4, 69.3)
- moved T1 1.55 mm to (127.5, 84.6)
- moved R4 1.19 mm to (109.0, 73.7)
- moved R3 0.39 mm to (109.0, 81.3)
Connections:
- J4 pad 1: unconnected-(J4-Pin_1-Pad1) -> GND
- J5 pad 1: unconnected-(J5-Pin_1-Pad1) -> GND
Routing:
- net Net-(J2-Pin_2): track 0.00 -> 37.5 mm
- net Net-(J2-Pin_1): track 0.00 -> 28.5 mm
- net Net-(J3-Pin_2): track 0.00 -> 14.0 mm
- net GND: track 0.00 -> 11.1 mm
- net Net-(J3-Pin_1): track 0.00 -> 8.92 mm
- net Net-(R1-Pad2): track 0.00 -> 8.38 mm
- net Net-(R2-Pad2): track 0.00 -> 7.94 mm
- net Net-(P2-Pad1): track 0.00 -> 3.17 mm
- net Net-(P1-Pad1): track 0.00 -> 3.17 mm
- added copper zone on B.Cu, net (none)
- added copper zone on F.Cu, net (none)
Other:
- outline, holes or cut-outs redrawn
