File: MRM5-Sensor/MRM5-Sensor.kicad_sch (KiCad schematic)
At the start: 12 parts, among them J1 1989447, J2 Conn_01x02_Socket, J3 Conn_01x02_Socket, J4 Conn_01x02_Socket, J5 Conn_01x02_Socket, P1 AC_L, P2 AC_N, T1 ZMPT107-1

Commit message: MRM5-tester added
Connections:
- net GND: now reaches J5.1 (Pin_1)
- net GND: now also J4.1 (Pin_1)
- no-connect marks 4 -> 2
Changed lines of the file:
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@@
+	)
+	(junction
+		(at 231.14 111.76)
+		(diameter 0)
+		(color 0 0 0 0)
 	)
 	(junction
@@
 		(at 240.03 104.14)
 	)
-	(no_connect
-		(at 240.03 101.6)
-	)
-	(no_connect
-		(at 240.03 111.76)
-	)
 	(wire
 		(pts
@@
 	(wire
 		(pts
+			(xy 231.14 111.76) (xy 240.03 111.76)
+		)
+		(stroke
+			(width 0)
+			(type default)
+		)
+	)
+	(wire
+		(pts
 			(xy 96.52 60.96) (xy 96.52 66.04)
 		)
@@
 	(wire
 		(pts
+			(xy 231.14 101.6) (xy 231.14 111.76)
+		)
+		(stroke
+			(width 0)
+			(type default)
+		)
+	)
+	(wire
+		(pts
 			(xy 167.64 128.27) (xy 167.64 138.43)
 		)
@@
 	(wire
 		(pts
+			(xy 231.14 116.84) (xy 231.14 111.76)
+		)
+		(stroke
+			(width 0)
+			(type default)
+		)
+	)
+	(wire
+		(pts
 			(xy 128.27 78.74) (xy 118.11 78.74)
 		)
@@
 		(pts
 			(xy 118.11 138.43) (xy 147.32 138.43)
+		)
+		(stroke
+			(width 0)
+			(type default)
+		)
+	)
+	(wire
+		(pts
+			(xy 240.03 101.6) (xy 231.14 101.6)
 		)
 		(stroke
@@
 					(unit 1)
 				)
+			)
+		)
+	)
+	(symbol
+		(lib_id "power:GND")
+		(at 231.14 116.84 0)
+		(unit 1)
+		(exclude_from_sim no)
+		(in_bom yes)
+		(on_board yes)
+		(dnp no)
+		(fields_autoplaced yes)
+		(property "Reference" "#PWR01"
+			(at 231.14 123.19 0)
+			(effects
+				(font
+					(size 1.27 1.27)
+				)
+				(hide yes)
+			)
+		)
+		(property "Value" "GND"
+			(at 231.14 121.92 0)
+			(effects
+				(font
+					(size 1.27 1.27)
+				)
+			)
+		)
+		(property "Footprint" ""
+			(at 231.14 116.84 0)
+			(effects
+				(font
+					(size 1.27 1.27)
+				)
+				(hide yes)
+			)
+		)
+		(property "Datasheet" ""
+			(at 231.14 116.84 0)
+			(effects
+				(font
+					(size 1.27 1.27)
+				)
+				(hide yes)
+			)
+		)
+		(property "Description" "Power symbol creates a global label with name \"GND\" , ground"
+			(at 231.14 116.84 0)
+			(effects
+				(font
+					(size 1.27 1.27)
+				)
+				(hide yes)
+			)
+		)
+		(pin "1"
+		)
+		(instances
+			(project ""
+				(path "/3a64da82-e1a5-468d-8721-80970913f271"
+					(reference "#PWR01")
+					(unit 1)
+				)

Commit message: MRM5-Sensor updated
Parts:
- removed J1: 1989447, 1989447, symbol Mouser:1989447
- removed J2, J3, J4, J5: Conn_01x02_Socket, Connector_PinSocket_2.54mm:PinSocket_1x02_P2.54mm_Vertical, symbol Connector:Conn_01x02_Socket
- removed P1: AC_L, Mouser:PAD_hole, symbol Mouser:PAD_hole2.6
- removed P2: AC_N, Mouser:PAD_hole, symbol Mouser:PAD_hole2.6
- removed R1, R2: 604k, PCM_Resistor_SMD_AKL:R_1206_3216Metric, symbol PCM_Resistor_AKL:R_1206
- removed R3: 5.49k, PCM_Resistor_SMD_AKL:R_0402_1005Metric, symbol PCM_Resistor_AKL:R_0402
- removed R4: 100, PCM_Resistor_SMD_AKL:R_0402_1005Metric, symbol PCM_Resistor_AKL:R_0402
- removed T1: ZMPT107-1, ZMPT1071, symbol Mouser:ZMPT107-1
Connections:
- no-connect marks 2 -> 0
Other:
- added sheet ethernet (ethernet.kicad_sch)
- added sheet mcu (mcu.kicad_sch)
