File: MRM5-tester/MRM5-tester (Copy).kicad_pcb (KiCad board)
At the start: 2 copper layers, 95 parts, among them IC1 STM32G051F8P6, IC2 OPA567AIRHGT, IC3 LD1085D2T33R, IC4 OPA567AIRHGT, J1 Conn_01x02, J2 Conn_01x02, J3 GSB1C41110SSHR, J4 PINHD_1x2_Female, J5 PINHD_1x2_Female, J6 Conn_01x05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

Commit message: case found!
Parts:
- moved C11 194.9 mm to (132.2, 109.0)
- moved C17 194.9 mm to (141.1, 107.1)
- moved C20 194.9 mm to (116.4, 89.1)
- moved C25 194.9 mm to (109.8, 100.5)
- moved C3 194.9 mm to (188.2, 113.0)
- moved FL1 194.9 mm to (130.8, 67.8)
- moved IC4 194.9 mm to (114.8, 103.8)
- moved J1 194.9 mm to (174.0, 104.0)
- moved J4 194.9 mm to (151.9, 99.8)
- moved J5 194.9 mm to (185.2, 99.8)
- moved P1 194.9 mm to (106.2, 67.0)
- moved P2 194.9 mm to (106.2, 90.1)
- moved P3 194.9 mm to (106.0, 119.5)
- moved P4 194.9 mm to (106.1, 103.4)
- moved PS1 194.9 mm to (153.2, 70.8)
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Routing:
- net GND: track 0.00 -> 614.8 mm, vias 0 -> 27
- net /analog/1V6: track 0.00 -> 320.9 mm, vias 0 -> 12
- net /analog/3V3: track 0.00 -> 244.8 mm, vias 0 -> 7
- net /interface/5V: track 0.00 -> 128.1 mm, vias 0 -> 3
- net /mcu/1V6_TFlag: track 0.00 -> 70.3 mm, vias 0 -> 2
- net Net-(U1-~{RXT}/GPIO.3): track 0.00 -> 64.8 mm
- net Net-(U1-~{TXT}/GPIO.2): track 0.00 -> 55.0 mm
- net /analog/Vn_h: track 0.00 -> 53.4 mm
- net /mcu/1V6_IFlag: track 0.00 -> 50.7 mm, vias 0 -> 2
- net /analog/V2p: track 0.00 -> 45.9 mm
- net Net-(Q1-B): track 0.00 -> 41.2 mm, vias 0 -> 2
- net /analog/Zfreed: track 0.00 -> 36.2 mm, vias 0 -> 1
- net /interface/UART_TXD: track 0.00 -> 33.7 mm, vias 0 -> 4
- net /analog/Z_TFlag: track 0.00 -> 30.4 mm, vias 0 -> 2
- net /interface/STLINK_RST: track 0.00 -> 28.6 mm, vias 0 -> 1
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- added copper zone on B.Cu, net /analog/1V6
- added copper zone on F.Cu, net /analog/1V6
- added copper zone on B.Cu, net GND
- added copper zone on F.Cu, net GND
Other:
- board outline added: 97 x 76.2 mm
