File: MRM5-tester/analog.kicad_sch (KiCad schematic)
At the start: 29 parts, among them IC2 OPA567AIRHGT, T1 ZMPT107-1, U2 ADA4528-2ACPZ

Commit message: MRM5-tester updated
Parts:
- D2: renamed from D9; footprint SOT95P240X120-3N -> Mouser:SOT95P240X120-3N
- R17: renamed from R15; value MBB02070C1004FCT00 -> 1MΩ 1W
- U2: value ADA4528-2ACPZ -> ADA4661-2ACPZ-RL
- renumbered C9 to C10, C22 to C11, C10 to C12, C11 to C13, C19 to C14, C12 to C15, C20 to C16, C13 to C17, C14 to C18, C21 to C9, R16 to R18, R17 to R19, R18 to R20, R19 to R21, R20 to R22, R21 to R23, R22 to R24, TP3 to TP2, TP2 to TP3
Changed lines of the file:
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@@
 			)
 		)
-		(property "Value" "ADA4528-2ACPZ"
+		(property "Value" "ADA4661-2ACPZ-RL"
 			(at 170.18 68.5486 0)
 			(effects
@@
 		(dnp no)
 		(fields_autoplaced yes)
-		(property "Reference" "C20"
+		(property "Reference" "C16"
 			(at 168.91 76.1999 0)
 			(effects
@@
 			(project "MRM5-tester"
 				(path "/6e775c75-0b09-4e5f-9bff-c5585ac94ad7/d46285ed-39e7-481d-bc83-4a7d1879f6d2"
-					(reference "C20")
+					(reference "C16")
 					(unit 1)
 				)
@@
 		(dnp no)
 		(fields_autoplaced yes)
-		(property "Reference" "R21"
+		(property "Reference" "R23"
 			(at 195.58 55.88 90)
 			(effects
@@
 			(project "MRM5-tester"
 				(path "/6e775c75-0b09-4e5f-9bff-c5585ac94ad7/d46285ed-39e7-481d-bc83-4a7d1879f6d2"
-					(reference "R21")
+					(reference "R23")
 					(unit 1)
 				)
@@
 		(dnp no)
 		(fields_autoplaced yes)
-		(property "Reference" "TP2"
+		(property "Reference" "TP3"
 			(at 256.54 56.3879 0)
 			(effects
@@
 			(project "MRM5-tester"
 				(path "/6e775c75-0b09-4e5f-9bff-c5585ac94ad7/d46285ed-39e7-481d-bc83-4a7d1879f6d2"
-					(reference "TP2")
+					(reference "TP3")
 					(unit 1)
 				)
@@
 		(dnp no)
 		(fields_autoplaced yes)
-		(property "Reference" "D9"
+		(property "Reference" "D2"
 			(at 100.33 24.13 90)
 			(effects
@@
 			)
 		)
-		(property "Footprint" "SOT95P240X120-3N"
+		(property "Footprint" "Mouser:SOT95P240X120-3N"
 			(at 196.52 15.24 0)
 			(effects
@@
 			(project ""
 				(path "/6e775c75-0b09-4e5f-9bff-c5585ac94ad7/d46285ed-39e7-481d-bc83-4a7d1879f6d2"
-					(reference "D9")
+					(reference "D2")
 					(unit 1)
 				)
@@
 		(dnp no)
 		(fields_autoplaced yes)
-		(property "Reference" "C21"
+		(property "Reference" "C9"
 			(at 137.16 54.6099 0)
 			(effects
@@
 			(project "MRM5-tester"
 				(path "/6e775c75-0b09-4e5f-9bff-c5585ac94ad7/d46285ed-39e7-481d-bc83-4a7d1879f6d2"
-					(reference "C21")
+					(reference "C9")
 					(unit 1)
 				)
@@
 		(dnp no)
 		(fields_autoplaced yes)
-		(property "Reference" "C22"
+		(property "Reference" "C11"
 			(at 147.32 54.6099 0)
 			(effects
@@
 			(project "MRM5-tester"
 				(path "/6e775c75-0b09-4e5f-9bff-c5585ac94ad7/d46285ed-39e7-481d-bc83-4a7d1879f6d2"
-					(reference "C22")
+					(reference "C11")
 					(unit 1)
 				)
@@
 		(dnp no)
 		(fields_autoplaced yes)
-		(property "Reference" "R20"
+		(property "Reference" "R22"
 			(at 182.88 55.88 90)
 			(effects
@@
 			(project "MRM5-tester"
 				(path "/6e775c75-0b09-4e5f-9bff-c5585ac94ad7/d46285ed-39e7-481d-bc83-4a7d1879f6d2"
-					(reference "R20")
+					(reference "R22")
 					(unit 1)
 				)
@@
 		(dnp no)
 		(fields_autoplaced yes)
-		(property "Reference" "TP3"
+		(property "Reference" "TP2"
 			(at 193.04 146.8119 0)
 			(effects
@@
 			(project "MRM5-tester"
 				(path "/6e775c75-0b09-4e5f-9bff-c5585ac94ad7/d46285ed-39e7-481d-bc83-4a7d1879f6d2"
-					(reference "TP3")
+					(reference "TP2")
 					(unit 1)
 				)
@@
 			)
 		)
-		(property "Value" "ADA4528-2ACPZ"
+		(property "Value" "ADA4661-2ACPZ-RL"
 			(at 229.87 72.39 0)
 			(effects
@@
 		(dnp no)
 		(fields_autoplaced yes)
-		(property "Reference" "C13"
+		(property "Reference" "C17"
 			(at 208.28 72.3899 0)
 			(effects
@@
 			(project "MRM5-tester"
 				(path "/6e775c75-0b09-4e5f-9bff-c5585ac94ad7/d46285ed-39e7-481d-bc83-4a7d1879f6d2"
-					(reference "C13")
+					(reference "C17")
 					(unit 1)
 				)
@@
 		(dnp no)
 		(fields_autoplaced yes)
-		(property "Reference" "R17"
+		(property "Reference" "R19"
 			(at 105.41 55.88 90)
 			(effects
@@
 			(project "MRM5-tester"
 				(path "/6e775c75-0b09-4e5f-9bff-c5585ac94ad7/d46285ed-39e7-481d-bc83-4a7d1879f6d2"
-					(reference "R17")
+					(reference "R19")
 					(unit 1)
 				)
@@
 		(dnp no)
 		(fields_autoplaced yes)
-		(property "Reference" "C10"
+		(property "Reference" "C12"
 			(at 147.32 107.9499 0)
 			(effects
@@
 			(project "MRM5-tester"
 				(path "/6e775c75-0b09-4e5f-9bff-c5585ac94ad7/d46285ed-39e7-481d-bc83-4a7d1879f6d2"
-					(reference "C10")
+					(reference "C12")
 					(unit 1)
 				)
@@
 		(dnp no)
 		(fields_autoplaced yes)
-		(property "Reference" "C11"
+		(property "Reference" "C13"
 			(at 153.67 39.37 90)
 			(effects
@@
 			(project "MRM5-tester"
 				(path "/6e775c75-0b09-4e5f-9bff-c5585ac94ad7/d46285ed-39e7-481d-bc83-4a7d1879f6d2"
-					(reference "C11")
+					(reference "C13")
 					(unit 1)
 				)
@@
 		(dnp no)
 		(fields_autoplaced yes)
-		(property "Reference" "R18"
+		(property "Reference" "R20"
 			(at 118.11 55.88 90)
 			(effects
@@
 			(project "MRM5-tester"
 				(path "/6e775c75-0b09-4e5f-9bff-c5585ac94ad7/d46285ed-39e7-481d-bc83-4a7d1879f6d2"
-					(reference "R18")
+					(reference "R20")
 					(unit 1)
 				)
@@
 		(dnp no)
 		(fields_autoplaced yes)
-		(property "Reference" "C9"
+		(property "Reference" "C10"
 			(at 140.97 162.5599 0)
 			(effects
@@
 			(project "MRM5-tester"
 				(path "/6e775c75-0b09-4e5f-9bff-c5585ac94ad7/d46285ed-39e7-481d-bc83-4a7d1879f6d2"
-					(reference "C9")
+					(reference "C10")
 					(unit 1)
 				)
@@
 		(dnp no)
 		(fields_autoplaced yes)
-		(property "Reference" "R22"
+		(property "Reference" "R24"
 			(at 203.2 121.92 90)
 			(effects
@@
 			(project "MRM5-tester"
 				(path "/6e775c75-0b09-4e5f-9bff-c5585ac94ad7/d46285ed-39e7-481d-bc83-4a7d1879f6d2"
-					(reference "R22")
+					(reference "R24")
 					(unit 1)
 				)
@@
 		(dnp no)
 		(fields_autoplaced yes)
-		(property "Reference" "R19"
+		(property "Reference" "R21"
 			(at 144.78 148.5899 0)
 			(effects
@@
 			(project "MRM5-tester"
 				(path "/6e775c75-0b09-4e5f-9bff-c5585ac94ad7/d46285ed-39e7-481d-bc83-4a7d1879f6d2"
-					(reference "R19")
+					(reference "R21")
 					(unit 1)
 				)
@@
 		(dnp no)
 		(fields_autoplaced yes)
-		(property "Reference" "R15"
+		(property "Reference" "R17"
 			(at 50.8 58.42 0)
 			(effects
@@
 			)
 		)
-		(property "Value" "MBB02070C1004FCT00"
+		(property "Value" "1MΩ 1W"
 			(at 50.8 60.96 0)
 			(effects
@@
 			(project "MRM5-tester"
 				(path "/6e775c75-0b09-4e5f-9bff-c5585ac94ad7/d46285ed-39e7-481d-bc83-4a7d1879f6d2"
-					(reference "R15")
+					(reference "R17")
 					(unit 1)
 				)
@@
 		(dnp no)
 		(fields_autoplaced yes)
-		(property "Reference" "C14"
+		(property "Reference" "C18"
 			(at 227.33 39.37 90)
 			(effects
@@
 			(project "MRM5-tester"
 				(path "/6e775c75-0b09-4e5f-9bff-c5585ac94ad7/d46285ed-39e7-481d-bc83-4a7d1879f6d2"
-					(reference "C14")
+					(reference "C18")
 					(unit 1)
 				)
@@
 		(dnp no)
 		(fields_autoplaced yes)
-		(property "Reference" "R16"
+		(property "Reference" "R18"
 			(at 99.06 69.8499 0)
 			(effects
@@
 			(project "MRM5-tester"
 				(path "/6e775c75-0b09-4e5f-9bff-c5585ac94ad7/d46285ed-39e7-481d-bc83-4a7d1879f6d2"
-					(reference "R16")
+					(reference "R18")
 					(unit 1)
 				)
@@
 		(dnp no)
 		(fields_autoplaced yes)
-		(property "Reference" "C12"
+		(property "Reference" "C15"
 			(at 160.02 109.2199 0)
 			(effects
@@
 			(project "MRM5-tester"
 				(path "/6e775c75-0b09-4e5f-9bff-c5585ac94ad7/d46285ed-39e7-481d-bc83-4a7d1879f6d2"
-					(reference "C12")
+					(reference "C15")
 					(unit 1)
 				)
@@
 		(dnp no)
 		(fields_autoplaced yes)
-		(property "Reference" "C19"
+		(property "Reference" "C14"
 			(at 158.75 76.1999 0)
 			(effects
@@
 			(project "MRM5-tester"
 				(path "/6e775c75-0b09-4e5f-9bff-c5585ac94ad7/d46285ed-39e7-481d-bc83-4a7d1879f6d2"
-					(reference "C19")
-					(unit 1)
-				)
+					(reference "C14")
+					(unit 1)
+				)

Commit message: case updated
Parts:
- added L1: 744770218, Mouser:WE-PD_744770218, symbol Mouser:744770218
Connections:
- net at P3.1: now also L1.2; no longer R24.2
- new net: L1.1, R24.2
Other:
- moved on the sheet: P3, P4
Changed lines of the file:
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@@
 	(wire
 		(pts
+			(xy 232.41 128.27) (xy 234.95 128.27)
+		)
+		(stroke
+			(width 0)
+			(type default)
+		)
+	)
+	(wire
+		(pts
 			(xy 109.22 30.48) (xy 114.3 30.48)
 		)
@@
 	(wire
 		(pts
-			(xy 203.2 139.7) (xy 223.52 139.7)
+			(xy 203.2 139.7) (xy 234.95 139.7)
 		)
 		(stroke
@@
 	(wire
 		(pts
-			(xy 207.01 128.27) (xy 223.52 128.27)
+			(xy 207.01 128.27) (xy 212.09 128.27)
 		)
 		(stroke
@@
 	(symbol
 		(lib_id "Mouser:PAD_hole2.6")
-		(at 224.79 128.27 0)
+		(at 236.22 128.27 0)
 		(mirror x)
 		(unit 1)
@@
 		(fields_autoplaced yes)
 		(property "Reference" "P3"
-			(at 226.06 124.46 0)
+			(at 237.49 124.46 0)
 			(effects
 				(font
@@
 		)
 		(property "Value" "~"
-			(at 226.06 127 0)
+			(at 237.49 127 0)
 			(effects
 				(font
@@
 		)
 		(property "Footprint" "Mouser:PAD_Hole_D2mm"
-			(at 224.79 125.984 0)
+			(at 236.22 125.984 0)
 			(effects
 				(font
@@
 		)
 		(property "Datasheet" ""
-			(at 224.79 128.27 0)
+			(at 236.22 128.27 0)
 			(effects
 				(font
@@
 		)
 		(property "Description" ""
-			(at 224.79 128.27 0)
+			(at 236.22 128.27 0)
 			(effects
 				(font
@@
 	(symbol
 		(lib_id "Mouser:PAD_hole2.6")
-		(at 224.79 139.7 0)
+		(at 236.22 139.7 0)
 		(mirror x)
 		(unit 1)
@@
 		(fields_autoplaced yes)
 		(property "Reference" "P4"
-			(at 226.06 135.89 0)
+			(at 237.49 135.89 0)
 			(effects
 				(font
@@
 		)
 		(property "Value" "~"
-			(at 226.06 138.43 0)
+			(at 237.49 138.43 0)
 			(effects
 				(font
@@
 		)
 		(property "Footprint" "Mouser:PAD_Hole_D2mm"
-			(at 224.79 137.414 0)
+			(at 236.22 137.414 0)
 			(effects
 				(font
@@
 		)
 		(property "Datasheet" ""
-			(at 224.79 139.7 0)
+			(at 236.22 139.7 0)
 			(effects
 				(font
@@
 		)
 		(property "Description" ""
-			(at 224.79 139.7 0)
+			(at 236.22 139.7 0)
 			(effects
 				(font
@@
 					(unit 1)
 				)
+			)
+		)
+	)
+	(symbol
+		(lib_id "Mouser:744770218")
+		(at 212.09 128.27 0)
+		(unit 1)
+		(exclude_from_sim no)
+		(in_bom yes)
+		(on_board yes)
+		(dnp no)
+		(fields_autoplaced yes)
+		(property "Reference" "L1"
+			(at 222.25 121.92 0)
+			(effects
+				(font
+					(size 1.27 1.27)
+				)
+			)
+		)
+		(property "Value" "744770218"
+			(at 222.25 124.46 0)
+			(effects
+				(font
+					(size 1.27 1.27)
+				)
+			)
+		)
+		(property "Footprint" "Mouser:WE-PD_744770218"
+			(at 228.6 224.46 0)
+			(effects
+				(font
+					(size 1.27 1.27)
+				)
+				(justify left top)
+				(hide yes)
+			)
+		)
+		(property "Datasheet" ""
+			(at 228.6 324.46 0)
+			(effects
+				(font
+					(size 1.27 1.27)
+				)
+				(justify left top)
+				(hide yes)
+			)
+		)
+		(property "Description" "Wurth WE-PD Series Shielded Wire-wound SMD Inductor 180 uH +/-20% 1.4A Idc"
+			(at 212.09 128.27 0)
+			(effects
+				(font
+					(size 1.27 1.27)
+				)
+				(hide yes)
+			)
+		)
+		(property "Height" ""
+			(at 228.6 524.46 0)
+			(effects
+				(font
+					(size 1.27 1.27)
+				)
+				(justify left top)
+				(hide yes)
+			)
+		)
+		(property "Manufacturer_Name" "Wurth Elektronik"
+			(at 228.6 624.46 0)
+			(effects
+				(font
+					(size 1.27 1.27)
+				)
+				(justify left top)
+				(hide yes)
+			)
+		)
+		(property "Manufacturer_Part_Number" "744770218"
+			(at 228.6 724.46 0)
+			(effects
+				(font
+					(size 1.27 1.27)
+				)
+				(justify left top)
+				(hide yes)
+			)
+		)
+		(property "Mouser Part Number" "710-744770218"
+			(at 228.6 824.46 0)
+			(effects
+				(font
+					(size 1.27 1.27)
+				)
+				(justify left top)
+				(hide yes)
+			)
+		)
+		(property "Mouser Price/Stock" "https://www.mouser.com/Search/Refine.aspx?Keyword=710-744770218"
+			(at 228.6 924.46 0)
+			(effects
+				(font
+					(size 1.27 1.27)
+				)
+				(justify left top)
+				(hide yes)
+			)
+		)
+		(property "Arrow Part Number" ""
+			(at 228.6 1024.46 0)
+			(effects
+				(font
+					(size 1.27 1.27)
+				)
+				(justify left top)
+				(hide yes)
+			)
+		)
+		(property "Arrow Price/Stock" ""
+			(at 228.6 1124.46 0)
+			(effects
+				(font
+					(size 1.27 1.27)
+				)
+				(justify left top)
+				(hide yes)
+			)
+		)
+		(pin "2"
+		)
+		(pin "1"
+		)
+		(instances
+			(project ""
+				(path "/6e775c75-0b09-4e5f-9bff-c5585ac94ad7/d46285ed-39e7-481d-bc83-4a7d1879f6d2"
+					(reference "L1")
+					(unit 1)
+				)

Commit message: tester pcb updated
Connections:
- net V2p: now reaches D2.3 (A/K), R18.2, R19.1, T1.3
Changed lines of the file:
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@@
+	)
+	(junction
+		(at 86.36 67.31)
+		(diameter 0)
+		(color 0 0 0 0)
 	)
 	(junction
@@
 	)
 	(junction
+		(at 86.36 64.77)
+		(diameter 0)
+		(color 0 0 0 0)
+	)
+	(junction
 		(at 190.5 128.27)
 		(diameter 0)
@@
 	(wire
 		(pts
+			(xy 86.36 67.31) (xy 88.9 67.31)
+		)
+		(stroke
+			(width 0)
+			(type default)
+		)
+	)
+	(wire
+		(pts
 			(xy 91.44 64.77) (xy 96.52 64.77)
 		)
@@
 		(pts
 			(xy 254 60.96) (xy 254 64.77)
+		)
+		(stroke
+			(width 0)
+			(type default)
+		)
+	)
+	(wire
+		(pts
+			(xy 86.36 62.23) (xy 86.36 64.77)
 		)
 		(stroke
@@
 		(shape input)
 		(at 162.56 52.07 0)
+		(fields_autoplaced yes)
+		(effects
+			(font
+				(size 1.27 1.27)
+			)
+			(justify left)
+		)
+	)
+	(hierarchical_label "V2p"
+		(shape input)
+		(at 86.36 62.23 90)
 		(fields_autoplaced yes)
 		(effects
@@
 		)
 	)
+	(hierarchical_label "V2n"
+		(shape input)
+		(at 88.9 67.31 0)
+		(fields_autoplaced yes)
+		(effects
+			(font
+				(size 1.27 1.27)
+			)
+			(justify left)
+		)
+	)

Commit message: case found!
Parts:
- C10, C12, C13, C14, C17, C18, C7, C9: footprint PCM_Capacitor_SMD_AKL:C_0402_1005Metric -> PCM_Capacitor_SMD_AKL:C_0603_1608Metric
- C11, C15, C16, C8: footprint PCM_Capacitor_SMD_AKL:C_0603_1608Metric -> PCM_Capacitor_SMD_AKL:C_1206_3216Metric
Changed lines of the file:
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@@
 			)
 		)
-		(property "Footprint" "PCM_Capacitor_SMD_AKL:C_0603_1608Metric"
+		(property "Footprint" "PCM_Capacitor_SMD_AKL:C_1206_3216Metric"
 			(at 127.9652 167.64 0)
 			(effects
@@
 			)
 		)
-		(property "Footprint" "PCM_Capacitor_SMD_AKL:C_0603_1608Metric"
+		(property "Footprint" "PCM_Capacitor_SMD_AKL:C_1206_3216Metric"
 			(at 166.0652 81.28 0)
 			(effects
@@
 			)
 		)
-		(property "Footprint" "PCM_Capacitor_SMD_AKL:C_0402_1005Metric"
+		(property "Footprint" "PCM_Capacitor_SMD_AKL:C_0603_1608Metric"
 			(at 132.3848 52.07 0)
 			(effects
@@
 			)
 		)
-		(property "Footprint" "PCM_Capacitor_SMD_AKL:C_0603_1608Metric"
+		(property "Footprint" "PCM_Capacitor_SMD_AKL:C_1206_3216Metric"
 			(at 144.4752 59.69 0)
 			(effects
@@
 			)
 		)
-		(property "Footprint" "PCM_Capacitor_SMD_AKL:C_0402_1005Metric"
+		(property "Footprint" "PCM_Capacitor_SMD_AKL:C_0603_1608Metric"
 			(at 203.5048 69.85 0)
 			(effects
@@
 			)
 		)
-		(property "Footprint" "PCM_Capacitor_SMD_AKL:C_0402_1005Metric"
+		(property "Footprint" "PCM_Capacitor_SMD_AKL:C_0603_1608Metric"
 			(at 122.2248 71.12 0)
 			(effects
@@
 			)
 		)
-		(property "Footprint" "PCM_Capacitor_SMD_AKL:C_0402_1005Metric"
+		(property "Footprint" "PCM_Capacitor_SMD_AKL:C_0603_1608Metric"
 			(at 142.5448 105.41 0)
 			(effects
@@
 			)
 		)
-		(property "Footprint" "PCM_Capacitor_SMD_AKL:C_0402_1005Metric"
+		(property "Footprint" "PCM_Capacitor_SMD_AKL:C_0603_1608Metric"
 			(at 157.48 46.0248 0)
 			(effects
@@
 			)
 		)
-		(property "Footprint" "PCM_Capacitor_SMD_AKL:C_0402_1005Metric"
+		(property "Footprint" "PCM_Capacitor_SMD_AKL:C_0603_1608Metric"
 			(at 136.1948 160.02 0)
 			(effects
@@
 			)
 		)
-		(property "Footprint" "PCM_Capacitor_SMD_AKL:C_0402_1005Metric"
+		(property "Footprint" "PCM_Capacitor_SMD_AKL:C_0603_1608Metric"
 			(at 231.14 46.0248 0)
 			(effects
@@
 			)
 		)
-		(property "Footprint" "PCM_Capacitor_SMD_AKL:C_0603_1608Metric"
+		(property "Footprint" "PCM_Capacitor_SMD_AKL:C_1206_3216Metric"
 			(at 157.1752 114.3 0)
 			(effects
@@
 			)
 		)
-		(property "Footprint" "PCM_Capacitor_SMD_AKL:C_0402_1005Metric"
+		(property "Footprint" "PCM_Capacitor_SMD_AKL:C_0603_1608Metric"
 			(at 153.9748 73.66 0)
 			(effects
