File: MRM5-tester/MRM5-tester.kicad_sch (KiCad schematic)
At the start: 0 parts

Commit message: updated
Other:
- sheet analog ports: added Vn_sh; removed Vn_h
- sheet power ports: added Vn_sh; removed none
Changed lines of the file:
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@@
 		(color 0 0 0 0)
 	)
-	(junction
-		(at 116.84 148.59)
-		(diameter 0)
-		(color 0 0 0 0)
-	)
 	(wire
 		(pts
@@
 	(wire
 		(pts
-			(xy 116.84 92.71) (xy 116.84 148.59)
-		)
-		(stroke
-			(width 0)
-			(type default)
-		)
-	)
-	(wire
-		(pts
 			(xy 88.9 156.21) (xy 193.04 156.21)
 		)
@@
 	(wire
 		(pts
-			(xy 88.9 148.59) (xy 116.84 148.59)
+			(xy 88.9 148.59) (xy 193.04 148.59)
 		)
 		(stroke
@@
 	(wire
 		(pts
+			(xy 88.9 119.38) (xy 116.84 119.38)
+		)
+		(stroke
+			(width 0)
+			(type default)
+		)
+	)
+	(wire
+		(pts
 			(xy 88.9 144.78) (xy 193.04 144.78)
 		)
@@
 	(wire
 		(pts
-			(xy 88.9 121.92) (xy 129.54 121.92)
+			(xy 88.9 123.19) (xy 129.54 123.19)
 		)
 		(stroke
@@
 	(wire
 		(pts
-			(xy 120.65 118.11) (xy 120.65 88.9)
+			(xy 120.65 116.84) (xy 120.65 88.9)
 		)
 		(stroke
@@
 	(wire
 		(pts
+			(xy 116.84 92.71) (xy 116.84 119.38)
+		)
+		(stroke
+			(width 0)
+			(type default)
+		)
+	)
+	(wire
+		(pts
 			(xy 88.9 96.52) (xy 113.03 96.52)
 		)
@@
 	(wire
 		(pts
-			(xy 116.84 148.59) (xy 193.04 148.59)
-		)
-		(stroke
-			(width 0)
-			(type default)
-		)
-	)
-	(wire
-		(pts
 			(xy 167.64 88.9) (xy 193.04 88.9)
 		)
@@
 	(wire
 		(pts
-			(xy 88.9 118.11) (xy 120.65 118.11)
+			(xy 88.9 116.84) (xy 120.65 116.84)
 		)
 		(stroke
@@
 		)
 		(pin "1V6_TFlag" input
-			(at 129.54 121.92 180)
+			(at 129.54 123.19 180)
 			(effects
 				(font
@@
 		)
 		(pin "1V6_TFlag" input
-			(at 88.9 121.92 0)
+			(at 88.9 123.19 0)
 			(effects
 				(font
@@
 		)
 		(pin "Vp_sh" input
-			(at 88.9 118.11 0)
+			(at 88.9 116.84 0)
 			(effects
 				(font
@@
 		(pin "GND_bot" bidirectional
 			(at 88.9 156.21 0)
+			(effects
+				(font
+					(size 1.27 1.27)
+				)
+				(justify right)
+			)
+		)
+		(pin "Vn_sh" input
+			(at 88.9 119.38 0)
 			(effects
 				(font
@@
 			)
 		)
-		(pin "Vn_h" input
-			(at 88.9 92.71 0)
-			(effects
-				(font
-					(size 1.27 1.27)
-				)
-				(justify right)
-			)
-		)
 		(pin "Vp_sh" input
 			(at 88.9 88.9 0)
@@
 			(effects
 				(font
+					(size 1.27 1.27)
+				)
+				(justify right)
+			)
+		)
+		(pin "Vn_sh" input
+			(at 88.9 92.71 0)
+			(effects
+				(font
