File: MRM5-tester/MRM5-tester.kicad_pcb (KiCad board)
At the start: 2 copper layers, 95 parts, among them IC1 STM32G051F8P6, IC2 OPA567AIRHGT, IC3 LD1085D2T33R, IC4 OPA567AIRHGT, J1 Conn_01x02, J2 Conn_01x02, J3 GSB1C41110SSHR, J4 PINHD_1x2_Female, J5 PINHD_1x2_Female, J6 Conn_01x05, J7 Conn_01x05, Q1 SMMBT3906LT3G, Q2 SMMBT3906LT3G, Q3 SMMBT3906LT3G, Q4 SMMBT3906LT3G, Q5 SMMBT3906LT3G, Q6 SMMBT3906LT3G, T1 ZMPT107-1, U1 CP2102N-A02-GQFN20, U2 ADA4661-2ACPZ-RL

Commit message: 전류 입력시의 경우를 고려한 회로 추가
Parts:
- added IC5: OPA388IDBVR, Mouser:SOT95P280X145-5N, B.Cu at (149.5, 165.3)
- added R28: 1k, PCM_Resistor_SMD_AKL:R_0402_1005Metric, B.Cu at (153.5, 164.2)
- added R29: 1k, PCM_Resistor_SMD_AKL:R_0402_1005Metric, B.Cu at (153.5, 166.4)
- added R30: 2.7k, PCM_Resistor_SMD_AKL:R_0402_1005Metric, B.Cu at (153.5, 168.5)
- added R31: 2.7k, PCM_Resistor_SMD_AKL:R_0402_1005Metric, B.Cu at (153.5, 170.6)
- added VR1: PTD902-2015K-C504, Mouser:PTD9022015KC504, F.Cu at (30.5, 60.1)
- added VR2: PTD901-1215K-B103, Mouser:PTD9011015FA203, F.Cu at (20.2, 136.7)
- C1, C10, C11, C12, C13, C14, C15, C16, C17, C18, C19, C2, C21, C22, C23, C24, C25, C3, C4, C5, C6, C7, C8, C9, D1, D2, IC1, IC2, IC3, IC4, J1, J2, J3, J4, J5, J6, J7, L1, P3, P4, Q1, Q2, Q3, Q4, Q5, Q6, R1, R10, R11, R12, R13, R14, R15, R16, R18, R2, R20, R21, R22, R23, R24, R25, R26, R27, R3, R4, R5, R6, R7, R8, R9, Symbol1, U1, U2: moved to B.Cu
- R19: value 12.7k -> 10k; moved to B.Cu
- TP1, TP2, TP3: moved to F.Cu
- moved C26 259.1 mm to (130.8, 62.8), turned to -90 degrees
- moved PS1 251.3 mm to (99.5, 105.4), turned to 90 degrees
- moved FL1 236.8 mm to (97.4, 128.4), turned to 90 degrees
- moved Q1 228.6 mm to (170.6, 59.7), turned to 180 degrees
- moved RT1 222.7 mm to (100.5, 146.3), turned to 90 degrees
- moved R17 221.0 mm to (106.7, 136.4), turned to 0 degrees
- moved R2 220.0 mm to (168.4, 68.8), turned to 180 degrees
- moved P1 219.4 mm to (100.3, 153.0), turned to 90 degrees
- moved C19 213.1 mm to (184.2, 58.6), turned to 180 degrees
- moved R4 208.1 mm to (168.4, 78.4), turned to 180 degrees
- moved J3 201.2 mm to (195.8, 56.6), turned to 0 degrees
- moved RV1 200.4 mm to (116.0, 150.4), turned to 180 degrees
- moved IC3 198.7 mm to (181.6, 72.9), turned to -90 degrees
- moved T1 198.4 mm to (129.1, 129.8)
- moved Q2 197.2 mm to (174.9, 80.8), turned to 180 degrees
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Connections:
- C3 pad 2: /interface/5V -> Net-(D1-L3)
- C4 pad 2: /interface/5V -> Net-(D1-L3)
- C8 pad 1: GND -> /analog/1V6
- C8 pad 2: /analog/1V6 -> GND
- D1 pad 4: /interface/5V -> Net-(D1-L3)
- D2 pad 3: /analog/V2p -> Net-(D2-A/K)
- J3 pad A4: /interface/5V -> Net-(D1-L3)
- J3 pad A9: /interface/5V -> Net-(D1-L3)
- R11 pad 2: /interface/5V -> Net-(D1-L3)
- R18 pad 2: /analog/V2p -> Net-(D2-A/K)
- R19 pad 1: /analog/V2p -> /analog/Signal_Input
- R9 pad 2: /interface/5V -> Net-(D1-L3)
- T1 pad 3: /analog/V2p -> Net-(D2-A/K)
- U1 pad 7: /interface/5V -> Net-(D1-L3)
Other:
- board outline added: 143.7 x 111 mm
- board text added: "[Interface] Voltage Input: High Voltage/220V Voltage Input: Low Voltage/3.3V Voltage/Current Output: 3.3V/1A USB: Waveform data output, condition setting, etc. LED Indicators: Power, TX/RX, Over-temperature 1, 2, Over-current 1, 2 [Function Definition] Generate output signals based on input signals Simply generate output signals"

Commit message: 케이스에 마춰서 제작 중
Parts:
- removed J1, J2: Conn_01x02, Connector_PinHeader_2.54mm:PinHeader_1x02_P2.54mm_Vertical
- removed J7: Conn_01x05, Connector_PinSocket_2.54mm:PinSocket_1x05_P2.54mm_Vertical
- added C27: 47u, PCM_Capacitor_SMD_AKL:C_1206_3216Metric, B.Cu at (94.6, 74.0)
- added J10: Conn_01x02, Connector_PinHeader_2.54mm:PinHeader_1x02_P2.54mm_Vertical, B.Cu at (144.0, 111.0)
- added J8: Conn_01x02, Connector_PinHeader_2.54mm:PinHeader_1x02_P2.54mm_Vertical, F.Cu at (176.2, 49.0)
- added J9: Conn_01x02, Connector_PinHeader_2.54mm:PinHeader_1x02_P2.54mm_Vertical, F.Cu at (216.6, 111.0)
- added SW1: TL3302AF260QG, Mouser:TL3302AF260QG, F.Cu at (95.6, 85.7)
- added SW2: TL3302AF260QG, Mouser:TL3302AF260QG, F.Cu at (101.4, 85.7)
- added SW3: TL3302AF260QG, Mouser:TL3302AF260QG, F.Cu at (107.2, 85.6)
- C1, C2, C21, C22, C23, C25, IC1, IC4, R25, R26, R27: moved to F.Cu
- J4, J5: value PINHD_1x2_Female -> Conn_01x02; footprint Connector_PinSocket_2.54mm:PinSocket_1x02_P2.54mm_Vertical -> Connector_PinHeader_2.54mm:PinHeader_1x02_P2.54mm_Vertical
- J6: value Conn_01x05 -> PINHD_2x5_Female; footprint Connector_PinSocket_2.54mm:PinSocket_1x05_P2.54mm_Vertical -> Connector_PinSocket_2.54mm:PinSocket_2x05_P2.54mm_Vertical; moved to F.Cu
- LED1, LED2, LED3, LED4, LED5, LED6, LED7: footprint PCM_LED_THT_AKL:LED_D5.0mm -> PCM_LED_SMD_Handsoldering_AKL:LED_1206_3216Metric
- VR1, VR2: moved to B.Cu
- moved VR2 140.1 mm to (143.0, 69.3)
- moved LED6 138.0 mm to (81.0, 110.5)
- moved LED4 137.7 mm to (81.0, 99.4)
- moved Symbol1 137.6 mm to (57.6, 96.2)
- moved LED5 137.5 mm to (81.0, 121.7), turned to 90 degrees
- moved LED1 137.4 mm to (81.0, 66.0)
- moved LED7 137.4 mm to (81.0, 132.8)
- moved LED2 137.4 mm to (81.0, 77.1)
- moved LED3 137.4 mm to (81.0, 88.3)
- moved VR1 116.8 mm to (143.1, 91.1), turned to 0 degrees
- moved J5 102.6 mm to (103.5, 49.0), turned to -90 degrees
- moved C1 102.4 mm to (99.5, 71.5), turned to 90 degrees
- moved C2 100.1 mm to (102.1, 71.5), turned to 90 degrees
- moved C25 99.8 mm to (126.2, 80.2), turned to 180 degrees
- moved C8 99.5 mm to (91.8, 94.2)
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Connections:
- C20 pad 2: /analog/Vp_sh -> Net-(C20-Pad2)
- D2 pad 3: Net-(D2-A/K) -> /analog/PT1
- FL1 pad 1: /analog/Vp_sh -> Net-(C20-Pad2)
- J6 pad 2: /interface/STLINK_RST -> GND
- J6 pad 3: /interface/STLINK_CLK -> /interface/STLINK_RST
- J6 pad 4: /interface/STLINK_DIO -> /interface/5V
- J6 pad 5: /analog/3V3 -> /interface/STLINK_CLK
- R17 pad 1: /analog/Vp_sh -> /analog/Vn_h
- R18 pad 2: Net-(D2-A/K) -> /analog/PT1
- R30 pad 2: Net-(D2-A/K) -> /analog/PT1
- RT1 pad 2: /analog/Vp_sh -> Net-(C20-Pad2)
- T1 pad 1: /analog/Vp_ssh -> /power/FL1_out1_sh
- T1 pad 2: /analog/Vn_h -> /analog/Vp_ssh
- T1 pad 3: Net-(D2-A/K) -> /analog/1V6
- T1 pad 4: /analog/1V6 -> /analog/PT1
Other:
- outline, holes or cut-outs redrawn
- board text added: "Bottom"
- board text added: "Top"

Commit message: pcb updated
Parts:
- moved J6 14.4 mm to (130.3, 75.0), turned to -90 degrees
- moved R9 10.8 mm to (134.5, 60.9)
- moved R11 10.8 mm to (134.5, 63.4)
- moved R10 10.8 mm to (134.5, 62.1)
- moved C4 10.8 mm to (132.6, 59.4)
- moved C5 10.1 mm to (128.3, 55.6)
- moved C6 10.1 mm to (128.3, 53.6)
- moved C22 8.70 mm to (121.0, 81.0)
- moved D1 8.55 mm to (124.8, 58.7)
- moved C3 8.55 mm to (122.4, 55.6)
- moved U1 7.66 mm to (127.5, 64.3)
- moved R25 5.29 mm to (123.4, 96.9)
- moved R26 5.29 mm to (126.9, 93.7)
- moved IC4 5.29 mm to (122.2, 91.2)
- moved R27 5.29 mm to (119.6, 97.5)
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
Commit message: 1차 마감
Parts:
- added J1: PJ-037AH, Mouser:PJ037AH, F.Cu at (195.8, 53.3)
- J4: moved to F.Cu
- J6: moved to B.Cu
- moved Symbol1 58.8 mm to (116.2, 90.8), turned to 180 degrees
- moved C27 6.53 mm to (90.9, 68.6)
- moved C24 6.35 mm to (91.7, 70.9)
- moved SW1 5.80 mm to (101.4, 85.6)
- moved SW2 5.80 mm to (95.6, 85.6)
- moved C25 4.30 mm to (129.8, 81.2)
- moved C21 3.91 mm to (129.8, 85.1), turned to 180 degrees
- moved TP3 3.37 mm to (119.7, 116.3)
- moved J6 2.65 mm to (130.2, 72.3), turned to 90 degrees
- moved C14 2.34 mm to (116.3, 113.2), turned to 0 degrees
- moved C2 2.05 mm to (101.0, 73.2)
- moved C1 1.75 mm to (99.1, 73.2)
- moved C11 1.02 mm to (130.3, 120.9)
- moved R27 0.86 mm to (119.0, 96.9)
- moved TP1 0.66 mm to (127.1, 116.3)
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Connections:
- net Net-(C20-Pad2) renamed /power/FL1_in1_sh
- C26 pad 1: /interface/5V -> /interface/5V_bot
- C26 pad 2: GND -> /interface/GND_bot
- J6 pad 3: /interface/STLINK_RST -> /interface/5V
- J6 pad 4: /interface/5V -> /interface/STLINK_RST
- J6 pad 5: /interface/STLINK_CLK -> /interface/UART_TXD
- J6 pad 6: /interface/UART_TXD -> /interface/STLINK_CLK
- J6 pad 7: /interface/STLINK_DIO -> /interface/UART_RXD
- J6 pad 8: /interface/UART_RXD -> /interface/STLINK_DIO
- J8 pad 1: GND -> /interface/GND_bot
- J8 pad 2: /interface/5V -> /interface/5V_bot
- J9 pad 1: /analog/1V6 -> /analog/PT1_bot
- J9 pad 2: /analog/PT1 -> /analog/PT2_bot
- PS1 pad 3: GND -> /interface/GND_bot
- PS1 pad 4: /interface/5V -> /interface/5V_bot
- T1 pad 3: /analog/1V6 -> /analog/PT2_bot
- T1 pad 4: /analog/PT1 -> /analog/PT1_bot
Routing:
- net GND: track 0.00 -> 508.5 mm, vias 0 -> 24
- net /analog/3V3: track 0.00 -> 291.5 mm, vias 0 -> 16
- net /analog/1V6: track 0.00 -> 288.6 mm, vias 0 -> 9
- net Net-(U1-~{RXT}/GPIO.3): track 0.00 -> 93.4 mm, vias 0 -> 2
- net Net-(U1-~{TXT}/GPIO.2): track 0.00 -> 79.3 mm, vias 0 -> 2
- net /mcu/1V6_TFlag: track 0.00 -> 70.8 mm, vias 0 -> 3
- net /analog/sigV: track 0.00 -> 61.1 mm, vias 0 -> 2
- net /interface/5V: track 0.00 -> 60.6 mm, vias 0 -> 1
- net /analog/V2p: track 0.00 -> 53.9 mm
- net Net-(D1-L3): track 0.00 -> 51.4 mm, vias 0 -> 4
- net /analog/Zfreed: track 0.00 -> 50.4 mm, vias 0 -> 4
- net /mcu/1V6_IFlag: track 0.00 -> 49.4 mm, vias 0 -> 3
- net /analog/Z_TFlag: track 0.00 -> 46.8 mm, vias 0 -> 3
- net /power/FL1_out1_sh: track 0.00 -> 46.1 mm
- net /interface/STLINK_RST: track 0.00 -> 45.2 mm, vias 0 -> 1
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- added copper zone on B.Cu, net /analog/1V6
- added copper zone on F.Cu, net /analog/1V6
- added copper zone on B.Cu, net /interface/GND_bot
- added copper zone on F.Cu, net /interface/GND_bot
- added copper zone on B.Cu, net GND
- added copper zone on F.Cu, net GND
Other:
- outline, holes or cut-outs redrawn
- board text added: "V"
- board text added: "Vf"
- board text added: "Z"

Commit message: PCB 제작 1차 마감
Parts:
- U2: value ADA4661-2ACPZ-RL -> ADA4500-2ACPZ
Routing:
- net /analog/Z_TFlag: track 46.8 -> 48.1 mm
- net /analog/Zfreed: track 50.4 -> 51.6 mm
- net GND: track 508.5 -> 509.6 mm

Commit message: firmware updated
Parts:
- moved R28 13.4 mm to (186.2, 112.0), turned to 0 degrees
- renumbered C9 to C10, C10 to C11, C11 to C12, C8 to C13, C13 to C14, C14 to C15, C27 to C23, C23 to C24, C24 to C25, C25 to C26, C26 to C27, C12 to C7, C7 to C8, C15 to C9, IC5 to IC3, IC3 to IC4, IC4 to IC5, J4 to J1, J10 to J2, J5 to J3, J6 to J4, J3 to J5, J9 to J6, J8 to J7, J1 to J8, R28 to R17, R29 to R18, R24 to R22, R22 to R23, R31 to R24, R23 to R25, R30 to R26, R18 to R27, R17 to R28, R25 to R29, R26 to R30, R27 to R31, TP2 to TP1, TP1 to TP2, VR2 to VR1, VR1 to VR2
Connections:
- C20 pad 1: /analog/Vn_h -> /interface/Vn_h
- FL1 pad 2: /analog/Vn_h -> /interface/Vn_h
- IC2 pad 13: /analog/1V6 -> unconnected-(IC2-EP-Pad13)
- IC5 pad 13: /analog/1V6 -> unconnected-(IC5-EP-Pad13)
- P2 pad 1: /analog/Vn_h -> /interface/Vn_h
- R28 pad 1: /analog/Vn_h -> /power/FL1_out2_sh
- RV1 pad 1: /analog/Vn_h -> /interface/Vn_h
Routing:
- net /interface/Vn_h: track 0.00 -> 42.8 mm
- net /analog/Vn_h: track 42.8 -> 0.00 mm
- net GND: track 509.6 -> 531.8 mm, vias 24 -> 26
- net /analog/1V6: track 288.6 -> 299.3 mm
- net /power/FL1_out2_sh: track 15.2 -> 22.6 mm
- net /analog/Vp_ssh: track 10.6 -> 8.86 mm

Commit message: tester updated
Routing:
- net /analog/3V3: track 291.6 -> 292.2 mm
Changed lines of the file:
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@@
+	)
+	(segment
+		(start 93.99375 73)
+		(end 92.475 71.48125)
+		(width 0.8)
+		(layer "B.Cu")
+		(net 2)
 	)
 	(segment
@@
 	)
 	(segment
-		(start 93.3 66.6)
-		(end 100.86 66.6)
-		(width 0.8)
-		(layer "B.Cu")
-		(net 2)
-	)
-	(segment
 		(start 97.1 73)
 		(end 111.2 73)
@@
 		(start 111.2 73)
 		(end 111.79 72.41)
-		(width 0.8)
-		(layer "B.Cu")
-		(net 2)
-	)
-	(segment
-		(start 92.475 70.5)
-		(end 92.475 67.425)
 		(width 0.8)
 		(layer "B.Cu")
@@
 	)
 	(segment
-		(start 97.1 73)
-		(end 94.975 73)
-		(width 0.8)
-		(layer "B.Cu")
-		(net 2)
-	)
-	(segment
 		(start 104.9 93.9)
 		(end 111 87.8)
@@
 	)
 	(segment
+		(start 92.475 71.48125)
+		(end 92.475 67.425)
+		(width 0.8)
+		(layer "B.Cu")
+		(net 2)
+	)
+	(segment
 		(start 86.7 76.6)
 		(end 86.2 76.1)
+		(width 0.8)
+		(layer "B.Cu")
+		(net 2)
+	)
+	(segment
+		(start 92.475 67.425)
+		(end 93.3 66.6)
 		(width 0.8)
 		(layer "B.Cu")
@@
 	)
 	(segment
+		(start 93.3 66.6)
+		(end 100.86 66.6)
+		(width 0.8)
+		(layer "B.Cu")
+		(net 2)
+	)
+	(segment
 		(start 98.9 94.45)
 		(end 98.9 94.8)
@@
 	)
 	(segment
-		(start 94.975 73)
-		(end 92.475 70.5)
-		(width 0.8)
-		(layer "B.Cu")
-		(net 2)
-	)
-	(segment
 		(start 135.6 100)
 		(end 135.25 100.35)
@@
 	)
 	(segment
+		(start 97.1 73)
+		(end 93.99375 73)
+		(width 0.8)
+		(layer "B.Cu")
+		(net 2)
+	)
+	(segment
 		(start 135.6 97.9)
 		(end 135.6 100)
@@
 	)
 	(segment
-		(start 92.475 67.425)
-		(end 93.3 66.6)
-		(width 0.8)
-		(layer "B.Cu")
-		(net 2)
-	)
-	(segment
 		(start 86.6 72.5)
 		(end 85.9 71.8)
@@
 	)
 	(segment
+		(start 124.4 69.5)
+		(end 116.105464 69.5)
+		(width 0.2)
+		(layer "F.Cu")
+		(net 16)
+	)
+	(segment
 		(start 126 67.9)
 		(end 124.4 69.5)
@@
 	)
 	(segment
-		(start 124.4 69.5)
-		(end 116.4 69.5)
+		(start 113.480464 72.125)
+		(end 111.638 72.125)
 		(width 0.2)
 		(layer "F.Cu")
@@
 	)
 	(segment
-		(start 116.4 69.5)
-		(end 113.775 72.125)
-		(width 0.2)
-		(layer "F.Cu")
-		(net 16)
-	)
-	(segment
-		(start 113.775 72.125)
-		(end 111.638 72.125)
+		(start 116.105464 69.5)
+		(end 113.480464 72.125)
 		(width 0.2)
 		(layer "F.Cu")
@@
 	)
 	(segment
+		(start 115.9 67.6)
+		(end 112.675 70.825)
+		(width 0.2)
+		(layer "F.Cu")
+		(net 17)
+	)
+	(segment
 		(start 121.5 67.6)
-		(end 116.2 67.6)
+		(end 115.9 67.6)
 		(width 0.2)
 		(layer "F.Cu")
@@
 	)
 	(segment
-		(start 112.975 70.825)
+		(start 112.675 70.825)
 		(end 111.638 70.825)
-		(width 0.2)
-		(layer "F.Cu")
-		(net 17)
-	)
-	(segment
-		(start 116.2 67.6)
-		(end 112.975 70.825)
 		(width 0.2)
 		(layer "F.Cu")
@@
 	)
 	(segment
-		(start 112.425 70.175)
-		(end 115.9 66.7)
+		(start 111.638 70.175)
+		(end 111.825 70.175)
 		(width 0.2)
 		(layer "F.Cu")
@@
 	)
 	(segment
-		(start 115.9 66.7)
-		(end 119.7 66.7)
-		(width 0.2)
-		(layer "F.Cu")
-		(net 19)
-	)
-	(segment
 		(start 122.4 66.7)
 		(end 119.7 66.7)
@@
 	)
 	(segment
-		(start 111.638 70.175)
-		(end 112.425 70.175)
+		(start 111.825 70.175)
+		(end 115.3 66.7)
+		(width 0.2)
+		(layer "F.Cu")
+		(net 19)
+	)
+	(segment
+		(start 115.3 66.7)
+		(end 119.7 66.7)
 		(width 0.2)
 		(layer "F.Cu")
@@
 	)
 	(segment
-		(start 116.5 68.3)
+		(start 116.26829 68.3)
 		(end 119.3 68.3)
 		(width 0.2)
@@
 	)
 	(segment
+		(start 113.09329 71.475)
+		(end 116.26829 68.3)
+		(width 0.2)
+		(layer "F.Cu")
+		(net 21)
+	)
+	(segment
 		(start 111.638 71.475)
-		(end 113.325 71.475)
-		(width 0.2)
-		(layer "F.Cu")
-		(net 21)
-	)
-	(segment
-		(start 113.325 71.475)
-		(end 116 68.8)
-		(width 0.2)
-		(layer "F.Cu")
-		(net 21)
-	)
-	(segment
-		(start 116 68.8)
-		(end 116.5 68.3)
-		(width 0.2)
-		(layer "F.Cu")
+		(end 113.09329 71.475)
+		(width 0.2)
+		(layer "F.Cu")
