File: MRM5-tester/power.kicad_sch (KiCad schematic)
At the start: 17 parts, among them IC3 LD1085D2T33R, IC4 OPA567AIRHGT

Commit message: case found!
Parts:
- C20: value B32922X2104K000 -> X2-15B( 0.1uF / 275V)
- C21, C25: footprint PCM_Capacitor_SMD_AKL:C_0402_1005Metric -> PCM_Capacitor_SMD_AKL:C_0603_1608Metric
- C22, C23: footprint PCM_Capacitor_SMD_AKL:C_0603_1608Metric -> PCM_Capacitor_SMD_AKL:C_1206_3216Metric
Changed lines of the file:
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@@
 			)
 		)
-		(property "Footprint" "PCM_Capacitor_SMD_AKL:C_0603_1608Metric"
+		(property "Footprint" "PCM_Capacitor_SMD_AKL:C_1206_3216Metric"
 			(at 141.9352 120.65 0)
 			(effects
@@
 			)
 		)
-		(property "Footprint" "PCM_Capacitor_SMD_AKL:C_0402_1005Metric"
+		(property "Footprint" "PCM_Capacitor_SMD_AKL:C_0603_1608Metric"
 			(at 162.8648 146.05 0)
 			(effects
@@
 			)
 		)
-		(property "Footprint" "PCM_Capacitor_SMD_AKL:C_0603_1608Metric"
+		(property "Footprint" "PCM_Capacitor_SMD_AKL:C_1206_3216Metric"
 			(at 153.3652 153.67 0)
 			(effects
@@
 			)
 		)
-		(property "Footprint" "PCM_Capacitor_SMD_AKL:C_0402_1005Metric"
+		(property "Footprint" "PCM_Capacitor_SMD_AKL:C_0603_1608Metric"
 			(at 129.8448 113.03 0)
 			(effects
@@
 			)
 		)
-		(property "Value" "B32922X2104K000"
+		(property "Value" "X2-15B( 0.1uF / 275V)"
 			(at 128.27 48.2599 90)
 			(effects

Commit message: 케이스에 마춰서 제작 중
Parts:
- added C27: 47u, PCM_Capacitor_SMD_AKL:C_1206_3216Metric, symbol PCM_Capacitor_AKL:C_0603
Connections:
- net FL1_out1_sh is gone; now on net Vp_sh: FL1.4, PS1.1 (AC_1)
- net 3V3: now also C27.1
- net GND: now also C27.2
- net Vp_sh: no longer C20.2, FL1.1, RT1.2
- new net: C20.2, FL1.1, RT1.2
Changed lines of the file:
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@@
 	)
 	(junction
-		(at 161.29 73.66)
+		(at 128.27 96.52)
 		(diameter 0)
 		(color 0 0 0 0)
 	)
 	(junction
-		(at 128.27 96.52)
+		(at 149.86 96.52)
 		(diameter 0)
 		(color 0 0 0 0)
@@
 	)
 	(junction
+		(at 161.29 73.66)
+		(diameter 0)
+		(color 0 0 0 0)
+	)
+	(junction
 		(at 152.4 139.7)
 		(diameter 0)
@@
 	)
 	(junction
+		(at 149.86 73.66)
+		(diameter 0)
+		(color 0 0 0 0)
+	)
+	(junction
 		(at 87.63 118.11)
 		(diameter 0)
@@
 	)
 	(junction
+		(at 162.56 35.56)
+		(diameter 0)
+		(color 0 0 0 0)
+	)
+	(junction
 		(at 92.71 35.56)
 		(diameter 0)
@@
 	(wire
 		(pts
+			(xy 149.86 96.52) (xy 161.29 96.52)
+		)
+		(stroke
+			(width 0)
+			(type default)
+		)
+	)
+	(wire
+		(pts
 			(xy 123.19 118.11) (xy 125.73 118.11)
 		)
@@
 	(wire
 		(pts
+			(xy 152.4 26.67) (xy 162.56 26.67)
+		)
+		(stroke
+			(width 0)
+			(type default)
+		)
+	)
+	(wire
+		(pts
 			(xy 107.95 125.73) (xy 107.95 106.68)
 		)
@@
 	(wire
 		(pts
-			(xy 128.27 96.52) (xy 161.29 96.52)
+			(xy 128.27 96.52) (xy 149.86 96.52)
 		)
 		(stroke
@@
 	(wire
 		(pts
-			(xy 146.05 73.66) (xy 161.29 73.66)
+			(xy 146.05 73.66) (xy 149.86 73.66)
 		)
 		(stroke
@@
 	(wire
 		(pts
-			(xy 161.29 73.66) (xy 166.37 73.66)
-		)
-		(stroke
-			(width 0)
-			(type default)
-		)
-	)
-	(wire
-		(pts
-			(xy 123.19 30.48) (xy 124.46 30.48)
+			(xy 162.56 26.67) (xy 162.56 35.56)
 		)
 		(stroke
@@
 	(wire
 		(pts
-			(xy 161.29 81.28) (xy 161.29 73.66)
+			(xy 149.86 81.28) (xy 149.86 73.66)
 		)
 		(stroke
@@
 	(wire
 		(pts
+			(xy 161.29 73.66) (xy 166.37 73.66)
+		)
+		(stroke
+			(width 0)
+			(type default)
+		)
+	)
+	(wire
+		(pts
 			(xy 125.73 162.56) (xy 130.81 162.56)
 		)
@@
 	(wire
 		(pts
-			(xy 124.46 30.48) (xy 124.46 35.56)
+			(xy 123.19 110.49) (xy 123.19 118.11)
 		)
 		(stroke
@@
 	(wire
 		(pts
-			(xy 123.19 110.49) (xy 123.19 118.11)
+			(xy 149.86 73.66) (xy 161.29 73.66)
 		)
 		(stroke
@@
 	(wire
 		(pts
-			(xy 161.29 88.9) (xy 161.29 96.52)
+			(xy 149.86 88.9) (xy 149.86 96.52)
 		)
 		(stroke
@@
 	(wire
 		(pts
+			(xy 161.29 88.9) (xy 161.29 96.52)
+		)
+		(stroke
+			(width 0)
+			(type default)
+		)
+	)
+	(wire
+		(pts
 			(xy 124.46 35.56) (xy 124.46 40.64)
 		)
@@
 	(wire
 		(pts
+			(xy 161.29 73.66) (xy 161.29 81.28)
+		)
+		(stroke
+			(width 0)
+			(type default)
+		)
+	)
+	(wire
+		(pts
 			(xy 196.85 35.56) (xy 218.44 35.56)
 		)
@@
 	(wire
 		(pts
-			(xy 158.75 35.56) (xy 168.91 35.56)
+			(xy 158.75 35.56) (xy 162.56 35.56)
 		)
 		(stroke
@@
 	(wire
 		(pts
+			(xy 162.56 35.56) (xy 168.91 35.56)
+		)
+		(stroke
+			(width 0)
+			(type default)
+		)
+	)
+	(wire
+		(pts
 			(xy 218.44 54.61) (xy 204.47 54.61)
 		)
@@
 	(hierarchical_label "Vp_sh"
 		(shape input)
-		(at 123.19 30.48 180)
+		(at 152.4 26.67 180)
 		(fields_autoplaced yes)
 		(effects
@@
 	)
 	(symbol
-		(lib_id "PCM_Capacitor_AKL:C_0603")
-		(at 161.29 85.09 0)
-		(unit 1)
-		(exclude_from_sim no)
-		(in_bom yes)
-		(on_board yes)
-		(dnp no)
-		(fields_autoplaced yes)
-		(property "Reference" "C24"
-			(at 165.1 83.8199 0)
-			(effects
-				(font
-					(size 1.27 1.27)
-				)
-				(justify left)
-			)
-		)
-		(property "Value" "10uF, 16V"
-			(at 165.1 86.3599 0)
-			(effects
-				(font
-					(size 1.27 1.27)
-				)
-				(justify left)
-			)
-		)
-		(property "Footprint" "PCM_Capacitor_SMD_AKL:C_0603_1608Metric"
-			(at 162.2552 88.9 0)
-			(effects
-				(font
-					(size 1.27 1.27)
-				)
-				(hide yes)
-			)
-		)
-		(property "Datasheet" "~"
-			(at 161.29 85.09 0)
-			(effects
-				(font
-					(size 1.27 1.27)
-				)
-				(hide yes)
-			)
-		)
-		(property "Description" "SMD 0603 MLCC capacitor, Alternate KiCad Library"
-			(at 161.29 85.09 0)
-			(effects
-				(font
-					(size 1.27 1.27)
-				)
-				(hide yes)
-			)
-		)
-		(pin "1"
-		)
-		(pin "2"
-		)
-		(instances
-			(project ""
-				(path "/6e775c75-0b09-4e5f-9bff-c5585ac94ad7/c69ac902-00f4-4f29-a9f3-8d3beb585abf"
-					(reference "C24")
-					(unit 1)
-				)
-			)
-		)
-	)
-	(symbol
 		(lib_id "ktw07182:SSHB10HS-R11100")
 		(at 149.86 38.1 0)
@@
 	(symbol
 		(lib_id "PCM_Capacitor_AKL:C_0603")
+		(at 149.86 85.09 0)
+		(unit 1)
+		(exclude_from_sim no)
+		(in_bom yes)
+		(on_board yes)
+		(dnp no)
+		(fields_autoplaced yes)
+		(property "Reference" "C27"
+			(at 153.67 83.8199 0)
+			(effects
+				(font
+					(size 1.27 1.27)
+				)
+				(justify left)
+			)
+		)
+		(property "Value" "47u"
+			(at 153.67 86.3599 0)
+			(effects
+				(font
+					(size 1.27 1.27)
+				)
+				(justify left)
+			)
+		)
+		(property "Footprint" "PCM_Capacitor_SMD_AKL:C_1206_3216Metric"
+			(at 150.8252 88.9 0)
+			(effects
+				(font
+					(size 1.27 1.27)
+				)
+				(hide yes)
+			)
+		)
+		(property "Datasheet" "~"
+			(at 149.86 85.09 0)
+			(effects
+				(font
+					(size 1.27 1.27)
+				)
+				(hide yes)
+			)
+		)
+		(property "Description" "SMD 0603 MLCC capacitor, Alternate KiCad Library"
+			(at 149.86 85.09 0)
+			(effects
+				(font
+					(size 1.27 1.27)
+				)
+				(hide yes)
+			)
+		)
+		(pin "1"
+		)
+		(pin "2"
+		)
+		(instances
+			(project "MRM5-tester"
+				(path "/6e775c75-0b09-4e5f-9bff-c5585ac94ad7/c69ac902-00f4-4f29-a9f3-8d3beb585abf"
+					(reference "C27")
+					(unit 1)
+				)
+			)
+		)
+	)
+	(symbol
+		(lib_id "PCM_Capacitor_AKL:C_0603")
 		(at 95.25 83.82 0)
 		(unit 1)
@@
 					(unit 1)
 				)
+			)
+		)
+	)
+	(symbol
+		(lib_id "PCM_Capacitor_AKL:C_0603")
+		(at 161.29 85.09 0)
+		(unit 1)
+		(exclude_from_sim no)
+		(in_bom yes)
+		(on_board yes)
+		(dnp no)
+		(fields_autoplaced yes)
+		(property "Reference" "C24"
+			(at 165.1 83.8199 0)
+			(effects
+				(font
+					(size 1.27 1.27)
+				)
+				(justify left)
+			)
+		)
+		(property "Value" "10uF, 16V"
+			(at 165.1 86.3599 0)
+			(effects
+				(font
+					(size 1.27 1.27)
+				)
+				(justify left)
+			)
+		)
+		(property "Footprint" "PCM_Capacitor_SMD_AKL:C_0603_1608Metric"
+			(at 162.2552 88.9 0)
+			(effects
+				(font
+					(size 1.27 1.27)
+				)
+				(hide yes)
+			)
+		)
+		(property "Datasheet" "~"
+			(at 161.29 85.09 0)
+			(effects
+				(font
+					(size 1.27 1.27)
+				)
+				(hide yes)
+			)
+		)
+		(property "Description" "SMD 0603 MLCC capacitor, Alternate KiCad Library"
+			(at 161.29 85.09 0)
+			(effects
+				(font
+					(size 1.27 1.27)
+				)
+				(hide yes)
+			)
+		)
+		(pin "1"
+		)
+		(pin "2"
+		)
+		(instances
+			(project "MRM5-tester"
+				(path "/6e775c75-0b09-4e5f-9bff-c5585ac94ad7/c69ac902-00f4-4f29-a9f3-8d3beb585abf"
+					(reference "C24")
+					(unit 1)
+				)

Commit message: 1차 마감
Connections:
- net 5V: no longer C26.1, PS1.4 (+V0)
- net GND: no longer C26.2, PS1.3 (-V0)
- net FL1_in1_sh: now reaches C20.2, FL1.1, RT1.2
- new net 5V_bot: C26.1, PS1.4 (+V0)
- new net GND_bot: C26.2, PS1.3 (-V0)
Changed lines of the file:
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@@
+		)
+	)
+	(label "FL1_in1_sh"
+		(at 124.46 35.56 0)
+		(fields_autoplaced yes)
+		(effects
+			(font
+				(size 1.27 1.27)
+			)
+			(justify left bottom)
 		)
 	)
@@
 		)
 	)
-	(hierarchical_label "GND"
+	(hierarchical_label "GND_bot"
 		(shape bidirectional)
 		(at 218.44 54.61 0)
@@
 		)
 	)
-	(hierarchical_label "GND"
-		(shape bidirectional)
-		(at 218.44 35.56 0)
-		(fields_autoplaced yes)
-		(effects
-			(font
-				(size 1.27 1.27)
-			)
-			(justify left)
-		)
-	)
 	(hierarchical_label "1V6_IFlag"
 		(shape input)
@@
 			)
 			(justify right)
+		)
+	)
+	(hierarchical_label "GND_bot"
+		(shape bidirectional)
+		(at 218.44 35.56 0)
+		(fields_autoplaced yes)
+		(effects
+			(font
+				(size 1.27 1.27)
+			)
+			(justify left)
 		)
 	)
@@
 		)
 	)
-	(hierarchical_label "5V"
+	(hierarchical_label "5V_bot"
 		(shape input)
 		(at 218.44 38.1 0)

Commit message: updated
Connections:
- net 1V6: no longer IC4.13 (EP)
- net FL1_out2_sh renamed Vn_sh
- no-connect marks 0 -> 1
Changed lines of the file:
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@@
-	)
-	(junction
-		(at 107.95 125.73)
-		(diameter 0)
-		(color 0 0 0 0)
 	)
 	(junction
@@
 	)
 	(junction
+		(at 162.56 40.64)
+		(diameter 0)
+		(color 0 0 0 0)
+	)
+	(junction
 		(at 87.63 118.11)
 		(diameter 0)
@@
 		(color 0 0 0 0)
 	)
+	(no_connect
+		(at 107.95 125.73)
+	)
 	(wire
 		(pts
@@
 	(wire
 		(pts
+			(xy 162.56 40.64) (xy 158.75 40.64)
+		)
+		(stroke
+			(width 0)
+			(type default)
+		)
+	)
+	(wire
+		(pts
 			(xy 143.51 138.43) (xy 148.59 138.43)
 		)
@@
 	(wire
 		(pts
-			(xy 107.95 125.73) (xy 107.95 106.68)
+			(xy 104.14 106.68) (xy 104.14 134.62)
 		)
 		(stroke
@@
 	(wire
 		(pts
+			(xy 162.56 46.99) (xy 162.56 40.64)
+		)
+		(stroke
+			(width 0)
+			(type default)
+		)
+	)
+	(wire
+		(pts
 			(xy 162.56 26.67) (xy 162.56 35.56)
 		)
@@
 	(wire
 		(pts
-			(xy 107.95 106.68) (xy 148.59 106.68)
+			(xy 104.14 106.68) (xy 148.59 106.68)
 		)
 		(stroke
@@
 	(wire
 		(pts
+			(xy 167.64 46.99) (xy 162.56 46.99)
+		)
+		(stroke
+			(width 0)
+			(type default)
+		)
+	)
+	(wire
+		(pts
 			(xy 87.63 118.11) (xy 91.44 118.11)
 		)
@@
 	(wire
 		(pts
-			(xy 163.83 40.64) (xy 158.75 40.64)
+			(xy 163.83 40.64) (xy 162.56 40.64)
 		)
 		(stroke
@@
 	(wire
 		(pts
+			(xy 104.14 134.62) (xy 107.95 134.62)
+		)
+		(stroke
+			(width 0)
+			(type default)
+		)
+	)
+	(wire
+		(pts
 			(xy 116.84 162.56) (xy 123.19 162.56)
 		)
@@
 		(pts
 			(xy 163.83 38.1) (xy 168.91 38.1)
-		)
-		(stroke
-			(width 0)
-			(type default)
-		)
-	)
-	(wire
-		(pts
-			(xy 107.95 134.62) (xy 107.95 125.73)
 		)
 		(stroke
@@
 		)
 	)
+	(hierarchical_label "Vn_sh"
+		(shape input)
+		(at 167.64 46.99 0)
+		(fields_autoplaced yes)
+		(effects
+			(font
+				(size 1.27 1.27)
+			)
+			(justify left)
+		)
+	)

Commit message: firmware updated
Parts:
- renumbered C27 to C23, C23 to C24, C24 to C25, C25 to C26, C26 to C27, IC3 to IC4, IC4 to IC5, R25 to R29, R26 to R30, R27 to R31
Changed lines of the file:
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@@
 		(dnp no)
 		(fields_autoplaced yes)
-		(property "Reference" "C25"
+		(property "Reference" "C26"
 			(at 167.64 148.5899 0)
 			(effects
@@
 			(project "MRM5-tester"
 				(path "/6e775c75-0b09-4e5f-9bff-c5585ac94ad7/c69ac902-00f4-4f29-a9f3-8d3beb585abf"
-					(reference "C25")
+					(reference "C26")
 					(unit 1)
 				)
@@
 		(dnp no)
 		(fields_autoplaced yes)
-		(property "Reference" "C23"
+		(property "Reference" "C24"
 			(at 156.21 148.5899 0)
 			(effects
@@
 			(project "MRM5-tester"
 				(path "/6e775c75-0b09-4e5f-9bff-c5585ac94ad7/c69ac902-00f4-4f29-a9f3-8d3beb585abf"
-					(reference "C23")
+					(reference "C24")
 					(unit 1)
 				)
@@
 		(dnp no)
 		(fields_autoplaced yes)
-		(property "Reference" "IC3"
+		(property "Reference" "IC4"
 			(at 128.27 66.04 0)
 			(effects
@@
 			(project ""
 				(path "/6e775c75-0b09-4e5f-9bff-c5585ac94ad7/c69ac902-00f4-4f29-a9f3-8d3beb585abf"
-					(reference "IC3")
+					(reference "IC4")
 					(unit 1)
 				)
@@
 		(dnp no)
 		(fields_autoplaced yes)
-		(property "Reference" "R27"
+		(property "Reference" "R31"
 			(at 133.35 152.3999 0)
 			(effects
@@
 			(project "MRM5-tester"
 				(path "/6e775c75-0b09-4e5f-9bff-c5585ac94ad7/c69ac902-00f4-4f29-a9f3-8d3beb585abf"
-					(reference "R27")
+					(reference "R31")
 					(unit 1)
 				)
@@
 		(dnp no)
 		(fields_autoplaced yes)
-		(property "Reference" "C27"
+		(property "Reference" "C23"
 			(at 153.67 83.8199 0)
 			(effects
@@
 			(project "MRM5-tester"
 				(path "/6e775c75-0b09-4e5f-9bff-c5585ac94ad7/c69ac902-00f4-4f29-a9f3-8d3beb585abf"
-					(reference "C27")
+					(reference "C23")
 					(unit 1)
 				)
@@
 		(dnp no)
 		(fields_autoplaced yes)
-		(property "Reference" "C24"
+		(property "Reference" "C25"
 			(at 165.1 83.8199 0)
 			(effects
@@
 			(project "MRM5-tester"
 				(path "/6e775c75-0b09-4e5f-9bff-c5585ac94ad7/c69ac902-00f4-4f29-a9f3-8d3beb585abf"
-					(reference "C24")
+					(reference "C25")
 					(unit 1)
 				)
@@
 		(dnp no)
 		(fields_autoplaced yes)
-		(property "Reference" "C26"
+		(property "Reference" "C27"
 			(at 208.28 44.4499 90)
 			(effects
@@
 			(project ""
 				(path "/6e775c75-0b09-4e5f-9bff-c5585ac94ad7/c69ac902-00f4-4f29-a9f3-8d3beb585abf"
-					(reference "C26")
+					(reference "C27")
 					(unit 1)
 				)
@@
 		(dnp no)
 		(fields_autoplaced yes)
-		(property "Reference" "IC4"
+		(property "Reference" "IC5"
 			(at 149.86 129.5714 0)
 			(effects
@@
 			(project "MRM5-tester"
 				(path "/6e775c75-0b09-4e5f-9bff-c5585ac94ad7/c69ac902-00f4-4f29-a9f3-8d3beb585abf"
-					(reference "IC4")
+					(reference "IC5")
 					(unit 1)
 				)
@@
 		(dnp no)
 		(fields_autoplaced yes)
-		(property "Reference" "R25"
+		(property "Reference" "R29"
 			(at 81.28 111.76 90)
 			(effects
@@
 			(project "MRM5-tester"
 				(path "/6e775c75-0b09-4e5f-9bff-c5585ac94ad7/c69ac902-00f4-4f29-a9f3-8d3beb585abf"
-					(reference "R25")
+					(reference "R29")
 					(unit 1)
 				)
@@
 		(dnp no)
 		(fields_autoplaced yes)
-		(property "Reference" "R26"
+		(property "Reference" "R30"
 			(at 95.25 111.76 90)
 			(effects
@@
 			(project "MRM5-tester"
 				(path "/6e775c75-0b09-4e5f-9bff-c5585ac94ad7/c69ac902-00f4-4f29-a9f3-8d3beb585abf"
-					(reference "R26")
-					(unit 1)
-				)
+					(reference "R30")
+					(unit 1)
+				)
